Commit message: Update

File: urdf/g1_29dof_no_hands.urdf (robot description, URDF)
Before this commit: robot g1_29dof, 42 links, 41 joints
Links:
- link left_tool_connector_link: geometry collision cylinder length=0.022 radius=0.0205; visual cylinder length=0.022 radius=0.0205
- link right_tool_connector_link: geometry collision cylinder length=0.022 radius=0.0205; visual cylinder length=0.022 radius=0.0205

Commit message: Update

File: urdf/g1_29dof_no_hands.urdf (robot description, URDF)
Before this commit: robot g1_29dof, 42 links, 41 joints
Links:
- link left_tool_connector_link: geometry collision mesh filename=package://g1_description/meshes/tool_connector_cyl_x.stl; visual mesh filename=package://g1_description/meshes/tool_connector_cyl_x.stl
- link right_tool_connector_link: geometry collision mesh filename=package://g1_description/meshes/tool_connector_cyl_x.stl; visual mesh filename=package://g1_description/meshes/tool_connector_cyl_x.stl

Commit message: Update

File: urdf/g1_29dof_no_hands.urdf (robot description, URDF)
Before this commit: robot g1_29dof, 42 links, 41 joints
Joints:
- joint left_tool_attach_joint: origin xyz=0.022 0 0 rpy=0 0 0 -> xyz=0.022 0 0 rpy=-1.5707963267948966 1.5707963267948966 0
- joint right_tool_attach_joint: origin xyz=0.022 0 0 rpy=0 0 0 -> xyz=0.022 0 0 rpy=1.5707963267948966 1.5707963267948966 0
